Commit message: Brrrrr

File: linorobot2_description/urdf/controllers/diff_drive.urdf.xacro (robot description, xacro)
@@ -17,5 +17,6 @@
         <publish_odom_tf>false</publish_odom_tf>
         <publish_wheel_tf>true</publish_wheel_tf>
-        <odometry_frame>odom</odometry_frame>
+        <odemetry_topic>/odom</odemetry_topic>
+        <odometry_frame>/odom</odometry_frame>
       </plugin>
     </gazebo>

File: linorobot2_description/urdf/mech/base.urdf.xacro (robot description, xacro)
@@ -3,4 +3,9 @@
   <xacro:macro name="base" params="length width height mass wheel_radius wheel_pos_z">
     <link name="base_footprint"/>
+      <!-- <joint name="base_joint" type="fixed">
+      <origin xyz="0 0 0" rpy="0 0 0"/>
+      <parent link="base_link"/>
+      <child link="base_footprint"/>
+      </joint> -->
     <link name="base_link">
       <visual>
