Commit message: Change: added namespacing

File: linorobot2_description/urdf/mech/base.urdf.xacro (robot description, xacro)
@@ -1,6 +1,6 @@
 <?xml version="1.0"?>
 <robot xmlns:xacro="http://ros.org/wiki/xacro">
-  <xacro:macro name="base" params="length width height mass wheel_radius wheel_pos_z">
-    <link name="base_footprint"/>
+  <xacro:macro name="base" params="length width height mass wheel_radius wheel_pos_z namespace">
+    <link name="${namespace+'_footprint'}"/>
     <link name="base_link">
       <visual>
@@ -40,5 +40,5 @@
     </gazebo>
     <joint name="base_to_footprint" type="fixed">
-      <parent link="base_footprint"/>
+      <parent link="${namespace+'_footprint'}"/>
       <child link="base_link"/>
       <origin xyz="0 0 ${wheel_radius - wheel_pos_z}" rpy="0 0 0"/>

File: linorobot2_description/urdf/mech/layer2.urdf.xacro (robot description, xacro)
@@ -1,5 +1,5 @@
 <?xml version="1.0"?>
 <robot xmlns:xacro="http://ros.org/wiki/xacro">
-  <xacro:macro name="layer2">
+  <xacro:macro name="layer2" params="namespace">
    <link name="layer_2">
       <visual>
@@ -12,5 +12,5 @@
     </link>
     <joint name="base_to_layer2" type="fixed">
-      <parent link="base_footprint"/>
+      <parent link="${namespace+'_footprint'}"/>
       <child link="layer_2"/>
       <origin xyz="0 0 ${(wheel_radius - wheel_pos_z)+0.07}" rpy="0 0 0"/>

File: linorobot2_description/urdf/mech/layer3.urdf.xacro (robot description, xacro)
@@ -1,5 +1,5 @@
 <?xml version="1.0"?>
 <robot xmlns:xacro="http://ros.org/wiki/xacro">
-  <xacro:macro name="layer3">
+  <xacro:macro name="layer3" params="namespace">
     <link name="layer_3">
       <visual>
@@ -12,5 +12,5 @@
     </link>
     <joint name="layer2_to_layer3" type="fixed">
-      <parent link="base_footprint"/>
+      <parent link="${namespace+'_footprint'}"/>
       <child link="layer_3"/>
       <origin xyz="0 0 ${(wheel_radius - wheel_pos_z)+0.14}" rpy="0 0 0"/>

File: linorobot2_description/urdf/robots/2wd.urdf.xacro (robot description, xacro)
@@ -18,7 +18,12 @@
     wheel_radius="${wheel_radius}"
     wheel_pos_z="${wheel_pos_z}"
+    namespace="$(arg prefix)"
 />
-  <xacro:layer2/>
-  <xacro:layer3/>
+  <xacro:layer2
+    namespace="$(arg prefix)"
+  />
+  <xacro:layer3
+    namespace="$(arg prefix)"
+  />
   <xacro:wheel
     side="left"

Commit message: Added namespace to robot description

File: linorobot2_description/urdf/mech/base.urdf.xacro (robot description, xacro)
@@ -2,6 +2,6 @@
 <robot xmlns:xacro="http://ros.org/wiki/xacro">
   <xacro:macro name="base" params="length width height mass wheel_radius wheel_pos_z namespace">
-    <link name="${namespace+'_footprint'}"/>
-    <link name="base_link">
+    <link name="${namespace}_footprint"/>
+    <link name="${namespace}_base_link">
       <visual>
         <origin xyz="-0.15 0.1 0" rpy="0 0 -1.57"/>
@@ -29,5 +29,5 @@
       </inertial>
     </link>
-    <gazebo reference="base_link">
+    <gazebo reference="${namespace}_base_link">
       <visual>
         <material>
@@ -39,7 +39,7 @@
       </visual>
     </gazebo>
-    <joint name="base_to_footprint" type="fixed">
-      <parent link="${namespace+'_footprint'}"/>
-      <child link="base_link"/>
+    <joint name="${namespace}_base_to_footprint" type="fixed">
+      <parent link="${namespace}_footprint"/>
+      <child link="${namespace}_base_link"/>
       <origin xyz="0 0 ${wheel_radius - wheel_pos_z}" rpy="0 0 0"/>
     </joint>

File: linorobot2_description/urdf/mech/caster_wheel.urdf.xacro (robot description, xacro)
@@ -1,5 +1,5 @@
 <?xml version="1.0"?>
 <robot xmlns:xacro="http://ros.org/wiki/xacro">
-  <xacro:macro name="caster_wheel" params="side mass base_length wheel_radius wheel_pos_z">
+  <xacro:macro name="caster_wheel" params="side mass base_length wheel_radius wheel_pos_z namespace">
     <xacro:property name="caster_wheel_radius" value="${(wheel_radius - wheel_pos_z) / 2}" />
     <xacro:if value="${side == 'front'}">
@@ -9,5 +9,5 @@
         <xacro:property name="caster_wheel_x" value="${-(base_length / 2) + caster_wheel_radius}" />
     </xacro:if>
-    <link name="${side}_caster_wheel_link">
+    <link name="${namespace}_${side}_caster_wheel_link">
       <visual>
         <origin xyz="0 0 0" rpy="0 0 0"/>
@@ -33,11 +33,11 @@
       </inertial>
     </link>
-    <gazebo reference="${side}_caster_wheel_link">
+    <gazebo reference="${namespace}_${side}_caster_wheel_link">
         <mu1>0.01</mu1>
         <mu2>0.01</mu2>
     </gazebo>
-    <joint name="${side}_caster_wheel_joint" type="fixed">
-      <parent link="base_link"/>
-      <child link="${side}_caster_wheel_link"/>
+    <joint name="${namespace}_${side}_caster_wheel_joint" type="fixed">
+      <parent link="${namespace}_base_link"/>
+      <child link="${namespace}_${side}_caster_wheel_link"/>
       <origin xyz="${caster_wheel_x} 0 -${caster_wheel_radius}" rpy="0 0 0"/>
     </joint>

File: linorobot2_description/urdf/mech/layer2.urdf.xacro (robot description, xacro)
@@ -2,5 +2,5 @@
 <robot xmlns:xacro="http://ros.org/wiki/xacro">
   <xacro:macro name="layer2" params="namespace">
-   <link name="layer_2">
+   <link name="${namespace + '_layer_2'}">
       <visual>
         <origin xyz="-0.15 0.1 0" rpy="0 0 -1.57"/>
@@ -11,7 +11,7 @@
       </visual>
     </link>
-    <joint name="base_to_layer2" type="fixed">
+    <joint name="${namespace + '_base_to_layer2'}" type="fixed">
       <parent link="${namespace+'_footprint'}"/>
-      <child link="layer_2"/>
+      <child link="${namespace + '_layer_2'}"/>
       <origin xyz="0 0 ${(wheel_radius - wheel_pos_z)+0.07}" rpy="0 0 0"/>
     </joint>

File: linorobot2_description/urdf/mech/layer3.urdf.xacro (robot description, xacro)
@@ -2,5 +2,5 @@
 <robot xmlns:xacro="http://ros.org/wiki/xacro">
   <xacro:macro name="layer3" params="namespace">
-    <link name="layer_3">
+    <link name="${namespace + '_layer_3'}">
       <visual>
         <origin xyz="-0.15 0.1 0" rpy="0 0 -1.57"/>
@@ -11,7 +11,7 @@
       </visual>
     </link>
-    <joint name="layer2_to_layer3" type="fixed">
+    <joint name="${namespace + '_base_to_layer3'}" type="fixed">
       <parent link="${namespace+'_footprint'}"/>
-      <child link="layer_3"/>
+      <child link="${namespace + '_layer_3'}"/>
       <origin xyz="0 0 ${(wheel_radius - wheel_pos_z)+0.14}" rpy="0 0 0"/>
     </joint>

File: linorobot2_description/urdf/mech/wheel.urdf.xacro (robot description, xacro)
@@ -1,6 +1,6 @@
 <?xml version="1.0"?>
 <robot xmlns:xacro="http://ros.org/wiki/xacro">
-  <xacro:macro name="wheel" params="side radius width pos_x pos_y pos_z mass">
-    <link name="${side}_wheel_link">
+  <xacro:macro name="wheel" params="side radius width pos_x pos_y pos_z mass namespace">
+    <link name="${namespace}_${side}_wheel_link">
       <visual>
         <origin xyz="0 0 0" rpy="${pi/2} 0 0"/>
@@ -26,5 +26,5 @@
       </inertial>
     </link>
-    <gazebo reference="${side}_wheel_link">
+    <gazebo reference="${namespace}_${side}_wheel_link">
       <visual>
         <material>
@@ -36,8 +36,8 @@
       </visual>
     </gazebo>
-    <joint name="${side}_wheel_joint" type="continuous">
+    <joint name="${namespace}_${side}_wheel_joint" type="continuous">
       <axis xyz="0 1 0" />
-      <parent link="base_link"/>
-      <child link="${side}_wheel_link"/>
+      <parent link="${namespace}_base_link"/>
+      <child link="${namespace}_${side}_wheel_link"/>
       <origin xyz="${pos_x} ${pos_y} ${pos_z}" rpy="0 0 0"/>
     </joint>

File: linorobot2_description/urdf/robots/2wd.urdf.xacro (robot description, xacro)
@@ -34,4 +34,5 @@
     pos_z="${wheel_pos_z}"
     mass="${wheel_mass}"
+    namespace="$(arg prefix)"
   />
   <xacro:wheel
@@ -43,4 +44,5 @@
     pos_z="${wheel_pos_z}"
     mass="${wheel_mass}"
+    namespace="$(arg prefix)"
   />
   <xacro:if value="${front_caster_wheel}">
@@ -51,4 +53,5 @@
       wheel_radius="${wheel_radius}"
       wheel_pos_z="${wheel_pos_z}"
+      namespace="$(arg prefix)"
     />
   </xacro:if>
@@ -60,13 +63,18 @@
       wheel_radius="${wheel_radius}"
       wheel_pos_z="${wheel_pos_z}"
+      namespace="$(arg prefix)"
     />
   </xacro:if>
-  <xacro:imu/>
-  <xacro:generic_laser>
-    <xacro:insert_block name="laser_pose" />
+  <xacro:imu
+    namespace="$(arg prefix)"
+  />
+  <xacro:generic_laser
+    namespace="$(arg prefix)"
+    >
+    <xacro:insert_block name="laser_pose" />origin
   </xacro:generic_laser>
-  <xacro:depth_sensor>
+  <!-- <xacro:depth_sensor>
     <xacro:insert_block name="depth_sensor_pose" />
-  </xacro:depth_sensor>
+  </xacro:depth_sensor> -->
   <xacro:diff_drive_controller
     wheel_separation="${wheel_pos_y * 2}"

File: linorobot2_description/urdf/sensors/generic_laser.urdf.xacro (robot description, xacro)
@@ -2,5 +2,5 @@
 <robot xmlns:xacro="http://ros.org/wiki/xacro">
   <xacro:include filename="$(find linorobot2_description)/urdf/sensors/laser.urdf.xacro" />
-  <xacro:macro name="generic_laser" params="*origin">
+  <xacro:macro name="generic_laser" params="*origin namespace">
     <xacro:laser
       update_rate="10"
@@ -10,8 +10,9 @@
       min_range="0.08"
       max_range="12.0"
-      frame_id="laser"
+      frame_id="${namespace}_laser"
       topic_name="scan"
+      namespace="${namespace}"
     >
-      <xacro:insert_block name="origin" />
+      <xacro:insert_block name="origin" />origin
     </xacro:laser>
   </xacro:macro>

File: linorobot2_description/urdf/sensors/imu.urdf.xacro (robot description, xacro)
@@ -1,11 +1,11 @@
 <robot xmlns:xacro="http://ros.org/wiki/xacro">
-  <xacro:macro name="imu">
-    <link name="imu_link"/>
-    <joint name="imu_to_base_link" type="fixed">
-      <parent link="base_link"/>
-      <child link="imu_link"/>
+  <xacro:macro name="imu" params="namespace">
+    <link name="${namespace}_imu_link"/>
+    <joint name="${namespace}_imu_to_base_link" type="fixed">
+      <parent link="${namespace}_base_link"/>
+      <child link="${namespace}_imu_link"/>
       <origin xyz="0 0 0" rpy="0 0 0"/>
     </joint>
-    <gazebo reference="imu_link">
+    <gazebo reference="${namespace}_imu_link">
       <gravity>true</gravity>
       <sensor name="imu_sensor" type="imu">

File: linorobot2_description/urdf/sensors/laser.urdf.xacro (robot description, xacro)
@@ -1,5 +1,5 @@
 <robot xmlns:xacro="http://ros.org/wiki/xacro">
   <xacro:property name="M_PI" value="3.1415926535897931" />
-  <xacro:macro name="laser" params="*origin update_rate ray_count min_angle max_angle min_range max_range frame_id topic_name">
+  <xacro:macro name="laser" params="*origin update_rate ray_count min_angle max_angle min_range max_range frame_id topic_name namespace">
     <link name="${frame_id}">
       <visual>
@@ -37,5 +37,5 @@
     </gazebo>
     <joint name="${frame_id}_to_base_link" type="fixed">
-      <parent link="base_link"/>
+      <parent link="${namespace}_base_link"/>
       <child link="${frame_id}"/>
       <xacro:insert_block name="origin" />

Commit message: Moved over working code

File: linorobot2_description/urdf/mech/base.urdf.xacro (robot description, xacro)
@@ -1,12 +1,12 @@
 <?xml version="1.0"?>
 <robot xmlns:xacro="http://ros.org/wiki/xacro">
-  <xacro:macro name="base" params="length width height mass wheel_radius wheel_pos_z namespace">
-    <link name="${namespace}_footprint"/>
-    <link name="${namespace}_base_link">
+  <xacro:macro name="base" params="length width height mass wheel_radius wheel_pos_z">
+    <link name="base_footprint"/>
+    <link name="base_link">
       <visual>
         <origin xyz="-0.15 0.1 0" rpy="0 0 -1.57"/>
         <geometry>
           <!--box size="${length} ${width} ${height}"/-->
-          <mesh scale="0.001 0.001 0.001" filename="file:///home/ubu/linorobot2_ws/src/linorobot2/linorobot2_description/meshes/layer_1_solidworks.STL"/>
+          <mesh scale="0.001 0.001 0.001" filename="file://~/linorobot2_ws/src/linorobot2/linorobot2_description/meshes/layer_1_solidworks.STL"/>
           <!-- <mesh filename="" scale="0.001 0.001 0.001"/> -->
         </geometry>
@@ -29,5 +29,5 @@
       </inertial>
     </link>
-    <gazebo reference="${namespace}_base_link">
+    <gazebo reference="base_link">
       <visual>
         <material>
@@ -39,7 +39,7 @@
       </visual>
     </gazebo>
-    <joint name="${namespace}_base_to_footprint" type="fixed">
-      <parent link="${namespace}_footprint"/>
-      <child link="${namespace}_base_link"/>
+    <joint name="base_to_footprint" type="fixed">
+      <parent link="base_footprint"/>
+      <child link="base_link"/>
       <origin xyz="0 0 ${wheel_radius - wheel_pos_z}" rpy="0 0 0"/>
     </joint>

File: linorobot2_description/urdf/mech/caster_wheel.urdf.xacro (robot description, xacro)
@@ -1,5 +1,5 @@
 <?xml version="1.0"?>
 <robot xmlns:xacro="http://ros.org/wiki/xacro">
-  <xacro:macro name="caster_wheel" params="side mass base_length wheel_radius wheel_pos_z namespace">
+  <xacro:macro name="caster_wheel" params="side mass base_length wheel_radius wheel_pos_z">
     <xacro:property name="caster_wheel_radius" value="${(wheel_radius - wheel_pos_z) / 2}" />
     <xacro:if value="${side == 'front'}">
@@ -9,5 +9,5 @@
         <xacro:property name="caster_wheel_x" value="${-(base_length / 2) + caster_wheel_radius}" />
     </xacro:if>
-    <link name="${namespace}_${side}_caster_wheel_link">
+    <link name="${side}_caster_wheel_link">
       <visual>
         <origin xyz="0 0 0" rpy="0 0 0"/>
@@ -33,11 +33,11 @@
       </inertial>
     </link>
-    <gazebo reference="${namespace}_${side}_caster_wheel_link">
+    <gazebo reference="${side}_caster_wheel_link">
         <mu1>0.01</mu1>
         <mu2>0.01</mu2>
     </gazebo>
-    <joint name="${namespace}_${side}_caster_wheel_joint" type="fixed">
-      <parent link="${namespace}_base_link"/>
-      <child link="${namespace}_${side}_caster_wheel_link"/>
+    <joint name="${side}_caster_wheel_joint" type="fixed">
+      <parent link="base_link"/>
+      <child link="${side}_caster_wheel_link"/>
       <origin xyz="${caster_wheel_x} 0 -${caster_wheel_radius}" rpy="0 0 0"/>
     </joint>

File: linorobot2_description/urdf/mech/layer2.urdf.xacro (robot description, xacro)
@@ -1,17 +1,17 @@
 <?xml version="1.0"?>
 <robot xmlns:xacro="http://ros.org/wiki/xacro">
-  <xacro:macro name="layer2" params="namespace">
-   <link name="${namespace + '_layer_2'}">
+  <xacro:macro name="layer2">
+   <link name="layer_2">
       <visual>
         <origin xyz="-0.15 0.1 0" rpy="0 0 -1.57"/>
         <geometry>
-          <mesh scale="0.001 0.001 0.001" filename="file:///home/ubu/linorobot2_ws/src/linorobot2/linorobot2_description/meshes/layer_2_solidworks.STL"/>
+          <mesh scale="0.001 0.001 0.001" filename="file://~/linorobot2_ws/src/linorobot2/linorobot2_description/meshes/layer_2_solidworks.STL"/>
         </geometry>
         <material name="Grey"/>
       </visual>
     </link>
-    <joint name="${namespace + '_base_to_layer2'}" type="fixed">
-      <parent link="${namespace+'_footprint'}"/>
-      <child link="${namespace + '_layer_2'}"/>
+    <joint name="base_to_layer2" type="fixed">
+      <parent link="base_footprint"/>
+      <child link="layer_2"/>
       <origin xyz="0 0 ${(wheel_radius - wheel_pos_z)+0.07}" rpy="0 0 0"/>
     </joint>

File: linorobot2_description/urdf/mech/layer3.urdf.xacro (robot description, xacro)
@@ -1,17 +1,17 @@
 <?xml version="1.0"?>
 <robot xmlns:xacro="http://ros.org/wiki/xacro">
-  <xacro:macro name="layer3" params="namespace">
-    <link name="${namespace + '_layer_3'}">
+  <xacro:macro name="layer3">
+    <link name="layer_3">
       <visual>
         <origin xyz="-0.15 0.1 0" rpy="0 0 -1.57"/>
         <geometry>
-          <mesh scale="0.001 0.001 0.001" filename="file:///home/ubu/linorobot2_ws/src/linorobot2/linorobot2_description/meshes/layer_3_solidworks.STL"/>
+          <mesh scale="0.001 0.001 0.001" filename="file://~/linorobot2_ws/src/linorobot2/linorobot2_description/meshes/layer_3_solidworks.STL"/>
         </geometry>
         <material name="Grey"/>
       </visual>
     </link>
-    <joint name="${namespace + '_base_to_layer3'}" type="fixed">
-      <parent link="${namespace+'_footprint'}"/>
-      <child link="${namespace + '_layer_3'}"/>
+    <joint name="base_to_layer3" type="fixed">
+      <parent link="base_footprint"/>
+      <child link="layer_3"/>
       <origin xyz="0 0 ${(wheel_radius - wheel_pos_z)+0.14}" rpy="0 0 0"/>
     </joint>

File: linorobot2_description/urdf/mech/wheel.urdf.xacro (robot description, xacro)
@@ -1,6 +1,6 @@
 <?xml version="1.0"?>
 <robot xmlns:xacro="http://ros.org/wiki/xacro">
-  <xacro:macro name="wheel" params="side radius width pos_x pos_y pos_z mass namespace">
-    <link name="${namespace}_${side}_wheel_link">
+  <xacro:macro name="wheel" params="side radius width pos_x pos_y pos_z mass">
+    <link name="${side}_wheel_link">
       <visual>
         <origin xyz="0 0 0" rpy="${pi/2} 0 0"/>
@@ -26,5 +26,5 @@
       </inertial>
     </link>
-    <gazebo reference="${namespace}_${side}_wheel_link">
+    <gazebo reference="${side}_wheel_link">
       <visual>
         <material>
@@ -36,8 +36,8 @@
       </visual>
     </gazebo>
-    <joint name="${namespace}_${side}_wheel_joint" type="continuous">
+    <joint name="${side}_wheel_joint" type="continuous">
       <axis xyz="0 1 0" />
-      <parent link="${namespace}_base_link"/>
-      <child link="${namespace}_${side}_wheel_link"/>
+      <parent link="base_link"/>
+      <child link="${side}_wheel_link"/>
       <origin xyz="${pos_x} ${pos_y} ${pos_z}" rpy="0 0 0"/>
     </joint>

File: linorobot2_description/urdf/robots/2wd.urdf.xacro (robot description, xacro)
@@ -18,12 +18,7 @@
     wheel_radius="${wheel_radius}"
     wheel_pos_z="${wheel_pos_z}"
-    namespace="$(arg prefix)"
 />
-  <xacro:layer2
-    namespace="$(arg prefix)"
-  />
-  <xacro:layer3
-    namespace="$(arg prefix)"
-  />
+  <xacro:layer2/>
+  <xacro:layer3/>
   <xacro:wheel
     side="left"
@@ -34,5 +29,4 @@
     pos_z="${wheel_pos_z}"
     mass="${wheel_mass}"
-    namespace="$(arg prefix)"
   />
   <xacro:wheel
@@ -44,5 +38,4 @@
     pos_z="${wheel_pos_z}"
     mass="${wheel_mass}"
-    namespace="$(arg prefix)"
   />
   <xacro:if value="${front_caster_wheel}">
@@ -53,5 +46,4 @@
       wheel_radius="${wheel_radius}"
       wheel_pos_z="${wheel_pos_z}"
-      namespace="$(arg prefix)"
     />
   </xacro:if>
@@ -63,13 +55,8 @@
       wheel_radius="${wheel_radius}"
       wheel_pos_z="${wheel_pos_z}"
-      namespace="$(arg prefix)"
     />
   </xacro:if>
-  <xacro:imu
-    namespace="$(arg prefix)"
-  />
-  <xacro:generic_laser
-    namespace="$(arg prefix)"
-    >
+  <xacro:imu/>
+  <xacro:generic_laser>
     <xacro:insert_block name="laser_pose" />origin
   </xacro:generic_laser>

File: linorobot2_description/urdf/sensors/generic_laser.urdf.xacro (robot description, xacro)
@@ -2,5 +2,5 @@
 <robot xmlns:xacro="http://ros.org/wiki/xacro">
   <xacro:include filename="$(find linorobot2_description)/urdf/sensors/laser.urdf.xacro" />
-  <xacro:macro name="generic_laser" params="*origin namespace">
+  <xacro:macro name="generic_laser" params="*origin">
     <xacro:laser
       update_rate="10"
@@ -10,7 +10,6 @@
       min_range="0.08"
       max_range="12.0"
-      frame_id="${namespace}_laser"
+      frame_id="laser"
       topic_name="scan"
-      namespace="${namespace}"
     >
       <xacro:insert_block name="origin" />origin

File: linorobot2_description/urdf/sensors/imu.urdf.xacro (robot description, xacro)
@@ -1,11 +1,11 @@
 <robot xmlns:xacro="http://ros.org/wiki/xacro">
-  <xacro:macro name="imu" params="namespace">
-    <link name="${namespace}_imu_link"/>
-    <joint name="${namespace}_imu_to_base_link" type="fixed">
-      <parent link="${namespace}_base_link"/>
-      <child link="${namespace}_imu_link"/>
+  <xacro:macro name="imu">
+    <link name="imu_link"/>
+    <joint name="imu_to_base_link" type="fixed">
+      <parent link="base_link"/>
+      <child link="imu_link"/>
       <origin xyz="0 0 0" rpy="0 0 0"/>
     </joint>
-    <gazebo reference="${namespace}_imu_link">
+    <gazebo reference="imu_link">
       <gravity>true</gravity>
       <sensor name="imu_sensor" type="imu">

File: linorobot2_description/urdf/sensors/laser.urdf.xacro (robot description, xacro)
@@ -1,5 +1,5 @@
 <robot xmlns:xacro="http://ros.org/wiki/xacro">
   <xacro:property name="M_PI" value="3.1415926535897931" />
-  <xacro:macro name="laser" params="*origin update_rate ray_count min_angle max_angle min_range max_range frame_id topic_name namespace">
+  <xacro:macro name="laser" params="*origin update_rate ray_count min_angle max_angle min_range max_range frame_id topic_name">
     <link name="${frame_id}">
       <visual>
@@ -37,5 +37,5 @@
     </gazebo>
     <joint name="${frame_id}_to_base_link" type="fixed">
-      <parent link="${namespace}_base_link"/>
+      <parent link="base_link"/>
       <child link="${frame_id}"/>
       <xacro:insert_block name="origin" />

Commit message: Fixed Base

File: linorobot2_description/urdf/mech/base.urdf.xacro (robot description, xacro)
@@ -5,8 +5,7 @@
     <link name="base_link">
       <visual>
-        <origin xyz="-0.15 0.1 0" rpy="0 0 -1.57"/>
+        <origin xyz="0 0 0" rpy="0 0 0"/>
         <geometry>
-          <!--box size="${length} ${width} ${height}"/-->
-          <mesh scale="0.001 0.001 0.001" filename="file://~/linorobot2_ws/src/linorobot2/linorobot2_description/meshes/layer_1_solidworks.STL"/>
+          <box size="${length} ${width} ${height}"/>
           <!-- <mesh filename="" scale="0.001 0.001 0.001"/> -->
         </geometry>
