Commit message: safe state, namespace in progress???

File: linorobot2_description/urdf/mech/base.urdf.xacro (robot description, xacro)
@@ -4,4 +4,16 @@
    wheel_radius wheel_pos_z base_origo_offset caster_diameter">
     <link name="base_link"/>
+    <link name="odom" />
+    <joint name="odom_to_base" type="fixed">
+        <parent link="odom"/>
+        <child link="base_link"/>
+        <origin xyz="0 0 0" rpy="0 0 0"/>
+    </joint>
+    <joint name="base_footprint_joint" type="fixed">
+        <parent link="base_link"/>
+        <child link="base_footprint"/>
+        <origin xyz="0 0 0" rpy="0 0 0"/>
+    </joint>
+    <link name="base_footprint"/>
     <joint name="chassis_joint" type="fixed">
         <parent link="base_link"/>
@@ -9,10 +21,4 @@
         <origin xyz="-0.105 0 0"/>
     </joint>
-      <joint name="base_footprint_joint" type="fixed">
-        <parent link="base_link"/>
-        <child link="base_footprint"/>
-        <origin xyz="0 0 0" rpy="0 0 0"/>
-    </joint>
-    <link name="base_footprint"/>
     <link name="chassis">
       <visual>

File: linorobot2_description/urdf/mech/caster_wheel.urdf.xacro (robot description, xacro)
@@ -37,5 +37,5 @@
     </gazebo>
     <joint name="${side}_caster_wheel_joint" type="fixed">
-      <parent link="chassis"/>
+      <parent link="base_link"/>
       <child link="${side}_caster_wheel_link"/>
       <origin xyz="${caster_wheel_x} 0 0" rpy="0 0 0"/>

File: linorobot2_description/urdf/sensors/imu.urdf.xacro (robot description, xacro)
@@ -1,2 +1,3 @@
+<?xml version="1.0"?>
 <robot xmlns:xacro="http://ros.org/wiki/xacro">
   <xacro:macro name="imu">
@@ -16,5 +17,5 @@
       <plugin filename="libgazebo_ros_imu_sensor.so" name="imu_plugin">
           <ros>
-            <remapping>~/out:=imu/data</remapping>
+            <remapping>~/out:=/imu/data</remapping>
           </ros>
           <topicName>imu/data</topicName>

Commit message: .

File: linorobot2_description/urdf/mech/base.urdf.xacro (robot description, xacro)
@@ -4,10 +4,4 @@
    wheel_radius wheel_pos_z base_origo_offset caster_diameter">
     <link name="base_link"/>
-    <link name="odom" />
-    <joint name="odom_to_base" type="fixed">
-        <parent link="odom"/>
-        <child link="base_link"/>
-        <origin xyz="0 0 0" rpy="0 0 0"/>
-    </joint>
     <joint name="base_footprint_joint" type="fixed">
         <parent link="base_link"/>
