Commit message: pretty bot

File: linorobot2_description/urdf/mech/layer2.urdf.xacro (robot description, xacro)
@@ -20,5 +20,5 @@
       <parent link="base_link"/>
       <child link="layer_2"/>
-      <origin xyz="0 0 ${(wheel_radius - wheel_pos_z)+0.07}" rpy="0 0 0"/>
+      <origin xyz="-0.10 0 ${(wheel_radius - wheel_pos_z)+0.07}" rpy="0 0 0"/>
     </joint>
   </xacro:macro>

File: linorobot2_description/urdf/sensors/laser.urdf.xacro (robot description, xacro)
@@ -4,5 +4,5 @@
     <link name="${frame_id}">
       <visual>
-        <origin xyz="0 0 0.095" rpy="0 0 0"/>
+        <origin xyz="-0.125 0 0.14" rpy="0 0 0"/>
         <geometry>
           <cylinder radius="0.0375" length="0.05"/>
