Commit message: Change laser yaw

File: linorobot2_description/urdf/2wd_properties.urdf.xacro (robot description, xacro)
@@ -15,5 +15,5 @@
   <xacro:property name="rear_caster_wheel" value="true" />
   <xacro:property name="laser_pose">
-    <origin xyz="0.12 0 0.33" rpy="0 0 0"/>
+    <origin xyz="0.12 0 0.33" rpy="0 0 90"/>
   </xacro:property>
   <xacro:property name="depth_sensor_pose">

Commit message: Changed laser yaw

File: linorobot2_description/urdf/2wd_properties.urdf.xacro (robot description, xacro)
@@ -15,5 +15,5 @@
   <xacro:property name="rear_caster_wheel" value="true" />
   <xacro:property name="laser_pose">
-    <origin xyz="0.12 0 0.33" rpy="0 0 90"/>
+    <origin xyz="0.12 0 0.33" rpy="0 0 1.57"/>
   </xacro:property>
   <xacro:property name="depth_sensor_pose">

Commit message: Changed laser pitch

File: linorobot2_description/urdf/2wd_properties.urdf.xacro (robot description, xacro)
@@ -15,5 +15,5 @@
   <xacro:property name="rear_caster_wheel" value="true" />
   <xacro:property name="laser_pose">
-    <origin xyz="0.12 0 0.33" rpy="0 0 1.57"/>
+    <origin xyz="0.12 0 0.33" rpy="0 3.14 1.57"/>
   </xacro:property>
   <xacro:property name="depth_sensor_pose">

Commit message: changed lidar yaw and inverted again

File: linorobot2_description/urdf/2wd_properties.urdf.xacro (robot description, xacro)
@@ -15,5 +15,5 @@
   <xacro:property name="rear_caster_wheel" value="true" />
   <xacro:property name="laser_pose">
-    <origin xyz="0.12 0 0.33" rpy="0 3.14 1.57"/>
+    <origin xyz="0.12 0 0.33" rpy="0 0 1.57"/>
   </xacro:property>
   <xacro:property name="depth_sensor_pose">

Commit message: Update 2wd_properties.urdf.xacro

File: linorobot2_description/urdf/2wd_properties.urdf.xacro (robot description, xacro)
@@ -15,5 +15,5 @@
   <xacro:property name="rear_caster_wheel" value="true" />
   <xacro:property name="laser_pose">
-    <origin xyz="0.12 0 0.33" rpy="0 0 1.57"/>
+    <origin xyz="0.12 0 0.33" rpy="0 0 4.71238898"/>
   </xacro:property>
   <xacro:property name="depth_sensor_pose">

Commit message: Changed urdf to fit polybot

File: linorobot2_description/urdf/2wd_properties.urdf.xacro (robot description, xacro)
@@ -5,15 +5,15 @@
   <xacro:property name="base_height" value="0.003" />
   <xacro:property name="base_mass" value="1" />
-  <xacro:property name="wheel_radius" value="0.045" />
+  <xacro:property name="wheel_radius" value="0.068" />
   <xacro:property name="wheel_width" value="0.01" />
   <xacro:property name="wheel_pos_x" value="0.0" />
   <xacro:property name="wheel_pos_y" value="0.13" />
-  <xacro:property name="wheel_pos_z" value="-0.03" />
+  <xacro:property name="wheel_pos_z" value="0.033" />
   <xacro:property name="wheel_mass" value=".1" />
   <xacro:property name="wheel_torque" value="20" />
-  <xacro:property name="front_caster_wheel" value="true" />
+  <xacro:property name="front_caster_wheel" value="false" />
   <xacro:property name="rear_caster_wheel" value="true" />
   <xacro:property name="laser_pose">
-    <origin xyz="0.12 0 0.33" rpy="0 0 4.71238898"/>
+    <origin xyz="-0.045 0 0" rpy="0 0 4.71238898"/>
   </xacro:property>
   <xacro:property name="depth_sensor_pose">

File: linorobot2_description/urdf/mech/base.urdf.xacro (robot description, xacro)
@@ -5,7 +5,8 @@
     <link name="base_link">
       <visual>
-        <origin xyz="0 0 0" rpy="0 0 0"/>
+        <origin xyz="-0.15 0.1 0" rpy="0 0 -1.57"/>
         <geometry>
-          <box size="${length} ${width} ${height}"/>
+          <!--box size="${length} ${width} ${height}"/-->
+          <mesh scale="0.001 0.001 0.001" filename="file:///home/ubu/linorobot2_ws/src/linorobot2/linorobot2_description/meshes/layer_1_solidworks.STL"/>
           <!-- <mesh filename="" scale="0.001 0.001 0.001"/> -->
         </geometry>

File: linorobot2_description/urdf/robots/2wd.urdf.xacro (robot description, xacro)
@@ -3,4 +3,6 @@
   <xacro:include filename="$(find linorobot2_description)/urdf/2wd_properties.urdf.xacro" />
   <xacro:include filename="$(find linorobot2_description)/urdf/mech/base.urdf.xacro" />
+  <xacro:include filename="$(find linorobot2_description)/urdf/mech/layer2.urdf.xacro" />
+  <xacro:include filename="$(find linorobot2_description)/urdf/mech/layer3.urdf.xacro" />
   <xacro:include filename="$(find linorobot2_description)/urdf/mech/wheel.urdf.xacro" />
   <xacro:include filename="$(find linorobot2_description)/urdf/mech/caster_wheel.urdf.xacro" />
@@ -17,4 +19,6 @@
     wheel_pos_z="${wheel_pos_z}"
 />
+  <xacro:layer2/>
+  <xacro:layer3/>
   <xacro:wheel
     side="left"

File: linorobot2_description/urdf/sensors/laser.urdf.xacro (robot description, xacro)
@@ -4,5 +4,5 @@
     <link name="${frame_id}">
       <visual>
-        <origin xyz="0 0 -0.025" rpy="0 0 0"/>
+        <origin xyz="0 0 0.095" rpy="0 0 0"/>
         <geometry>
           <cylinder radius="0.0375" length="0.05"/>

Commit message: 2nd urdf iteration

File: linorobot2_description/urdf/2wd_properties.urdf.xacro (robot description, xacro)
@@ -1,13 +1,16 @@
 <?xml version="1.0"?>
 <robot xmlns:xacro="http://ros.org/wiki/xacro">
-  <xacro:property name="base_length" value="0.24" />
-  <xacro:property name="base_width" value="0.275" />
-  <xacro:property name="base_height" value="0.003" />
+  <xacro:property name="base_length" value="0.40" />
+  <xacro:property name="base_width" value="0.30" />
+  <xacro:property name="base_height" value="0.0062" />
   <xacro:property name="base_mass" value="1" />
-  <xacro:property name="wheel_radius" value="0.068" />
-  <xacro:property name="wheel_width" value="0.01" />
-  <xacro:property name="wheel_pos_x" value="0.0" />
+  <xacro:property name="layer2_length" value="0.35"/>
+  <xacro:property name="layer2_width" value="0.25"/>
+  <xacro:property name="layer2_height" value="0.0062"/>
+  <xacro:property name="wheel_radius" value="0.0475" />
+  <xacro:property name="wheel_width" value="0.014" />
+  <xacro:property name="wheel_pos_x" value="0.150" />
   <xacro:property name="wheel_pos_y" value="0.13" />
-  <xacro:property name="wheel_pos_z" value="0.033" />
+  <xacro:property name="wheel_pos_z" value="-0.03" />
   <xacro:property name="wheel_mass" value=".1" />
   <xacro:property name="wheel_torque" value="20" />
@@ -15,8 +18,8 @@
   <xacro:property name="rear_caster_wheel" value="true" />
   <xacro:property name="laser_pose">
-    <origin xyz="-0.045 0 0" rpy="0 0 4.71238898"/>
+    <origin xyz="0 0 0.075" rpy="0 0 0"/>
   </xacro:property>
-  <xacro:property name="depth_sensor_pose">
+  <!-- <xacro:property name="depth_sensor_pose">
     <origin xyz="0.14 0.0 0.045" rpy="0 0 0"/>
-  </xacro:property>
+  </xacro:property> -->
 </robot>

File: linorobot2_description/urdf/mech/layer2.urdf.xacro (robot description, xacro)
@@ -1,13 +1,19 @@
 <?xml version="1.0"?>
 <robot xmlns:xacro="http://ros.org/wiki/xacro">
-  <xacro:macro name="layer2">
+  <xacro:macro name="layer2" params="length width height mass wheel_radius wheel_pos_z">
    <link name="layer_2">
       <visual>
-        <origin xyz="-0.15 0.1 0" rpy="0 0 -1.57"/>
+        <origin xyz="-0.015 0.1 0" rpy="0 0 0"/>
         <geometry>
-          <mesh scale="0.001 0.001 0.001" filename="file://~/linorobot2_ws/src/linorobot2/linorobot2_description/meshes/layer_2_solidworks.STL"/>
+          <box size="${length} ${width} ${height}"/>
         </geometry>
         <material name="Grey"/>
       </visual>
+      <collision>
+        <origin xyz="-0.015 0 0" rpy="0 0 0"/>
+        <geometry>
+          <box size="${length} ${width} ${height}"/>
+        </geometry>
+      </collision>
     </link>
     <joint name="base_to_layer2" type="fixed">

File: linorobot2_description/urdf/robots/2wd.urdf.xacro (robot description, xacro)
@@ -18,7 +18,13 @@
     wheel_radius="${wheel_radius}"
     wheel_pos_z="${wheel_pos_z}"
-/>
-  <xacro:layer2/>
-  <xacro:layer3/>
+  />
+  <xacro:layer2
+    length="${layer2_length}"
+    width="${layer2_width}"
+    height="${layer2_height}"
+    mass="${base_mass}"
+    wheel_radius="${wheel_radius}"
+    wheel_pos_z="${wheel_pos_z}"
+  />
   <xacro:wheel
     side="left"

File: linorobot2_description/urdf/sensors/laser.urdf.xacro (robot description, xacro)
@@ -1,2 +1,3 @@
+<?xml version="1.0"?>
 <robot xmlns:xacro="http://ros.org/wiki/xacro">
   <xacro:property name="M_PI" value="3.1415926535897931" />

Commit message: 3rd iteration urdf

File: linorobot2_description/urdf/2wd_properties.urdf.xacro (robot description, xacro)
@@ -18,5 +18,5 @@
   <xacro:property name="rear_caster_wheel" value="true" />
   <xacro:property name="laser_pose">
-    <origin xyz="0 0 0.075" rpy="0 0 0"/>
+    <origin xyz="0 0 0.0075" rpy="0 0 0"/>
   </xacro:property>
   <!-- <xacro:property name="depth_sensor_pose">

File: linorobot2_description/urdf/mech/layer2.urdf.xacro (robot description, xacro)
@@ -4,5 +4,5 @@
    <link name="layer_2">
       <visual>
-        <origin xyz="-0.015 0.1 0" rpy="0 0 0"/>
+        <origin xyz="0 -0.0015 0" rpy="0 0 0"/>
         <geometry>
           <box size="${length} ${width} ${height}"/>
@@ -11,5 +11,5 @@
       </visual>
       <collision>
-        <origin xyz="-0.015 0 0" rpy="0 0 0"/>
+        <origin xyz="0 -0.0015 0" rpy="0 0 0"/>
         <geometry>
           <box size="${length} ${width} ${height}"/>

Commit message: Update 2wd_properties.urdf.xacro

File: linorobot2_description/urdf/2wd_properties.urdf.xacro (robot description, xacro)
@@ -18,5 +18,5 @@
   <xacro:property name="rear_caster_wheel" value="true" />
   <xacro:property name="laser_pose">
-    <origin xyz="0 0 0.0075" rpy="0 0 0"/>
+    <origin xyz="0 0.125 0.0075" rpy="0 0 0"/>
   </xacro:property>
   <!-- <xacro:property name="depth_sensor_pose">

Commit message: REEEE

File: linorobot2_description/urdf/2wd_properties.urdf.xacro (robot description, xacro)
@@ -18,5 +18,5 @@
   <xacro:property name="rear_caster_wheel" value="true" />
   <xacro:property name="laser_pose">
-    <origin xyz="0 0.125 0.0075" rpy="0 0 0"/>
+    <origin xyz="0.125 0 0.0062" rpy="0 0 0"/>
   </xacro:property>
   <!-- <xacro:property name="depth_sensor_pose">

Commit message: Initial COmmit

File: linorobot2_description/urdf/2wd_properties.urdf.xacro (robot description, xacro)
@@ -5,9 +5,12 @@
   <xacro:property name="base_height" value="0.003" />
   <xacro:property name="base_mass" value="1" />
-  <xacro:property name="wheel_radius" value="0.068" />
+  <xacro:property name="layer2_length" value="0.35"/>
+  <xacro:property name="layer2_width" value="0.25"/>
+  <xacro:property name="layer2_height" value="0.0062"/>
+  <xacro:property name="wheel_radius" value="0.0475" />
   <xacro:property name="wheel_width" value="0.01" />
   <xacro:property name="wheel_pos_x" value="0.0" />
   <xacro:property name="wheel_pos_y" value="0.13" />
-  <xacro:property name="wheel_pos_z" value="0.033" />
+  <xacro:property name="wheel_pos_z" value="0" />
   <xacro:property name="wheel_mass" value=".1" />
   <xacro:property name="wheel_torque" value="20" />

File: linorobot2_description/urdf/controllers/diff_drive.urdf.xacro (robot description, xacro)
@@ -12,5 +12,5 @@
         <wheel_diameter>${wheel_radius * 2}</wheel_diameter>
         <max_wheel_acceleration>1.0</max_wheel_acceleration>
-        <robot_base_frame>base_footprint</robot_base_frame>
+        <robot_base_frame>base_link</robot_base_frame>
         <publish_odom>true</publish_odom>
         <publish_odom_tf>false</publish_odom_tf>

File: linorobot2_description/urdf/mech/base.urdf.xacro (robot description, xacro)
@@ -2,12 +2,21 @@
 <robot xmlns:xacro="http://ros.org/wiki/xacro">
   <xacro:macro name="base" params="length width height mass wheel_radius wheel_pos_z">
+    <link name="base_link"/>
+    <joint name="chassis_joint" type="fixed">
+        <parent link="base_link"/>
+        <child link="chassis"/>
+        <origin xyz="0.105 0 0"/>
+    </joint>
+      <joint name="base_footprint_joint" type="fixed">
+        <parent link="base_link"/>
+        <child link="base_footprint"/>
+        <origin xyz="0 0 0" rpy="0 0 0"/>
+    </joint>
     <link name="base_footprint"/>
-    <link name="base_link">
+    <link name="chassis">
       <visual>
-        <origin xyz="-0.15 0.1 0" rpy="0 0 -1.57"/>
+        <origin xyz="${length/2} 0 ${wheel_radius - wheel_pos_z}" rpy="0 0 0"/>
         <geometry>
-          <!--box size="${length} ${width} ${height}"/-->
-          <mesh scale="0.001 0.001 0.001" filename="file://~/linorobot2_ws/src/linorobot2/linorobot2_description/meshes/layer_1_solidworks.STL"/>
-          <!-- <mesh filename="" scale="0.001 0.001 0.001"/> -->
+          <box size="${length} ${width} ${height}"/>
         </geometry>
         <material name="yellow">
@@ -39,9 +48,4 @@
       </visual>
     </gazebo>
-    <joint name="base_to_footprint" type="fixed">
-      <parent link="base_footprint"/>
-      <child link="base_link"/>
-      <origin xyz="0 0 ${wheel_radius - wheel_pos_z}" rpy="0 0 0"/>
-    </joint>
   </xacro:macro>
 </robot>

File: linorobot2_description/urdf/mech/caster_wheel.urdf.xacro (robot description, xacro)
@@ -38,5 +38,5 @@
     </gazebo>
     <joint name="${side}_caster_wheel_joint" type="fixed">
-      <parent link="base_link"/>
+      <parent link="chassis"/>
       <child link="${side}_caster_wheel_link"/>
       <origin xyz="${caster_wheel_x} 0 -${caster_wheel_radius}" rpy="0 0 0"/>

File: linorobot2_description/urdf/mech/layer2.urdf.xacro (robot description, xacro)
@@ -1,16 +1,22 @@
 <?xml version="1.0"?>
 <robot xmlns:xacro="http://ros.org/wiki/xacro">
-  <xacro:macro name="layer2">
+  <xacro:macro name="layer2" params="length width height mass wheel_radius wheel_pos_z">
    <link name="layer_2">
       <visual>
-        <origin xyz="-0.15 0.1 0" rpy="0 0 -1.57"/>
+        <origin xyz="0 -0.0015 0" rpy="0 0 0"/>
         <geometry>
-          <mesh scale="0.001 0.001 0.001" filename="file://~/linorobot2_ws/src/linorobot2/linorobot2_description/meshes/layer_2_solidworks.STL"/>
+          <box size="${length} ${width} ${height}"/>
         </geometry>
         <material name="Grey"/>
       </visual>
+      <collision>
+        <origin xyz="0 -0.0015 0" rpy="0 0 0"/>
+        <geometry>
+          <box size="-${length} ${width} ${height}"/>
+        </geometry>
+      </collision>
     </link>
     <joint name="base_to_layer2" type="fixed">
-      <parent link="base_footprint"/>
+      <parent link="base_link"/>
       <child link="layer_2"/>
       <origin xyz="0 0 ${(wheel_radius - wheel_pos_z)+0.07}" rpy="0 0 0"/>

File: linorobot2_description/urdf/robots/2wd.urdf.xacro (robot description, xacro)
@@ -19,6 +19,12 @@
     wheel_pos_z="${wheel_pos_z}"
 />
-  <xacro:layer2/>
-  <xacro:layer3/>
+  <xacro:layer2
+    length="${layer2_length}"
+    width="${layer2_width}"
+    height="${layer2_height}"
+    mass="${base_mass}"
+    wheel_radius="${wheel_radius}"
+    wheel_pos_z="${wheel_pos_z}"
+  />
   <xacro:wheel
     side="left"

Commit message: Revamp IN progress

File: linorobot2_description/urdf/2wd_properties.urdf.xacro (robot description, xacro)
@@ -1,25 +1,27 @@
 <?xml version="1.0"?>
 <robot xmlns:xacro="http://ros.org/wiki/xacro">
-  <xacro:property name="base_length" value="0.24" />
-  <xacro:property name="base_width" value="0.275" />
-  <xacro:property name="base_height" value="0.003" />
+  <xacro:property name="base_length" value="0.40" />
+  <xacro:property name="base_width" value="0.30" />
+  <xacro:property name="base_height" value="0.0062" />
   <xacro:property name="base_mass" value="1" />
   <xacro:property name="layer2_length" value="0.35"/>
   <xacro:property name="layer2_width" value="0.25"/>
   <xacro:property name="layer2_height" value="0.0062"/>
+  <xacro:property name="base_origo" value="0.1" />
   <xacro:property name="wheel_radius" value="0.0475" />
-  <xacro:property name="wheel_width" value="0.01" />
-  <xacro:property name="wheel_pos_x" value="0.0" />
+  <xacro:property name="wheel_width" value="0.014" />
+  <xacro:property name="wheel_pos_x" value="0" />
   <xacro:property name="wheel_pos_y" value="0.13" />
   <xacro:property name="wheel_pos_z" value="0" />
   <xacro:property name="wheel_mass" value=".1" />
   <xacro:property name="wheel_torque" value="20" />
+  <xacro:property name="caster_diameter" value ="0.079"/>
   <xacro:property name="front_caster_wheel" value="false" />
   <xacro:property name="rear_caster_wheel" value="true" />
   <xacro:property name="laser_pose">
-    <origin xyz="-0.045 0 0" rpy="0 0 4.71238898"/>
+    <origin xyz="0.125 0 0.0062" rpy="0 0 0"/>
   </xacro:property>
-  <xacro:property name="depth_sensor_pose">
+  <!-- <xacro:property name="depth_sensor_pose">
     <origin xyz="0.14 0.0 0.045" rpy="0 0 0"/>
-  </xacro:property>
+  </xacro:property> -->
 </robot>

File: linorobot2_description/urdf/mech/base.urdf.xacro (robot description, xacro)
@@ -1,10 +1,11 @@
 <?xml version="1.0"?>
 <robot xmlns:xacro="http://ros.org/wiki/xacro">
-  <xacro:macro name="base" params="length width height mass wheel_radius wheel_pos_z">
+  <xacro:macro name="base" params="length width height mass
+   wheel_radius wheel_pos_z base_origo_offset caster_diameter">
     <link name="base_link"/>
     <joint name="chassis_joint" type="fixed">
         <parent link="base_link"/>
         <child link="chassis"/>
-        <origin xyz="0.105 0 0"/>
+        <origin xyz="-0.105 0 0"/>
     </joint>
       <joint name="base_footprint_joint" type="fixed">
@@ -16,5 +17,5 @@
     <link name="chassis">
       <visual>
-        <origin xyz="${length/2} 0 ${wheel_radius - wheel_pos_z}" rpy="0 0 0"/>
+        <origin xyz="0 0 ${caster_diameter/2}" rpy="0 0 0"/>
         <geometry>
           <box size="${length} ${width} ${height}"/>
@@ -33,7 +34,7 @@
         <origin xyz="0 0 0" rpy="0 0 0"/>
         <mass value="${mass}"/>
-        <inertia ixx="${(1/12) * mass * ((width  * width)  + (height * height))}" ixy="0.0" ixz="0.0"
-                 iyy="${(1/12) * mass * ((length * length) + (height * height))}" iyz="0.0"
-                 izz="${(1/12) * mass * ((length * length) + (width  * width))}"/>
+        <inertia ixx="${(1/12) * mass * (width  * 2 + height * 2)}" ixy="0.0" ixz="0.0"
+                 iyy="${(1/12) * mass * (length * 2 + height * 2)}" iyz="0.0"
+                 izz="${(1/12) * mass * (length * 2 + width * 2)}"/>
       </inertial>
     </link>

File: linorobot2_description/urdf/mech/caster_wheel.urdf.xacro (robot description, xacro)
@@ -1,11 +1,10 @@
 <?xml version="1.0"?>
 <robot xmlns:xacro="http://ros.org/wiki/xacro">
-  <xacro:macro name="caster_wheel" params="side mass base_length wheel_radius wheel_pos_z">
-    <xacro:property name="caster_wheel_radius" value="${(wheel_radius - wheel_pos_z) / 2}" />
+  <xacro:macro name="caster_wheel" params="side mass length caster_wheel_radius wheel_pos_z">
     <xacro:if value="${side == 'front'}">
-        <xacro:property name="caster_wheel_x" value="${(base_length / 2) - caster_wheel_radius}" />
+        <xacro:property name="caster_wheel_x" value="${( length / 2) - caster_wheel_radius}" />
     </xacro:if>
     <xacro:if value="${side == 'rear'}">
-        <xacro:property name="caster_wheel_x" value="${-(base_length / 2) + caster_wheel_radius}" />
+        <xacro:property name="caster_wheel_x" value="${-( length / 2) + caster_wheel_radius}" />
     </xacro:if>
     <link name="${side}_caster_wheel_link">
@@ -40,5 +39,5 @@
       <parent link="chassis"/>
       <child link="${side}_caster_wheel_link"/>
-      <origin xyz="${caster_wheel_x} 0 -${caster_wheel_radius}" rpy="0 0 0"/>
+      <origin xyz="${caster_wheel_x} 0 0" rpy="0 0 0"/>
     </joint>
   </xacro:macro>

File: linorobot2_description/urdf/robots/2wd.urdf.xacro (robot description, xacro)
@@ -12,18 +12,20 @@
   <xacro:include filename="$(find linorobot2_description)/urdf/controllers/diff_drive.urdf.xacro" />
   <xacro:base
-    length="${base_length}"
-    width="${base_width}"
-    height="${base_height}"
-    mass="${base_mass}"
-    wheel_radius="${wheel_radius}"
-    wheel_pos_z="${wheel_pos_z}"
+    length        = "${base_length}"
+    width         = "${base_width}"
+    height        = "${base_height}"
+    mass          = "${base_mass}"
+    wheel_radius  = "${wheel_radius}"
+    wheel_pos_z   = "${wheel_pos_z}"
+    base_origo_offset   = "${base_origo}"
+    caster_diameter     = "${caster_diameter}"
 />
   <xacro:layer2
-    length="${layer2_length}"
-    width="${layer2_width}"
-    height="${layer2_height}"
-    mass="${base_mass}"
-    wheel_radius="${wheel_radius}"
-    wheel_pos_z="${wheel_pos_z}"
+    length        = "${layer2_length}"
+    width         = "${layer2_width}"
+    height        = "${layer2_height}"
+    mass          = "${base_mass}"
+    wheel_radius  = "${wheel_radius}"
+    wheel_pos_z   = "${wheel_pos_z}"
   />
   <xacro:wheel
@@ -58,6 +60,6 @@
       side="rear"
       mass="0.01"
-      base_length="${base_length}"
-      wheel_radius="${wheel_radius}"
+      length="${base_length}"
+      caster_wheel_radius="${caster_diameter/2}"
       wheel_pos_z="${wheel_pos_z}"
     />
