Commit message: Revert "Merge branch 'Polygon-Generation' into One-big-simulation"
This reverts commit a067007681a2743c2e9a45f746fe557c2f6e826d, reversing
changes made to ac43001d0796424688f738b8d812c4fc38b0ff49.

File: linorobot2_description/urdf/2wd_properties.urdf.xacro (robot description, xacro)
@@ -1,7 +1,4 @@
 <?xml version="1.0"?>
 <robot xmlns:xacro="http://ros.org/wiki/xacro">
-  <xacro:property name="base_length" value="0.40" />
-  <xacro:property name="base_width" value="0.30" />
-  <xacro:property name="base_height" value="0.0062" />
   <xacro:property name="base_length" value="0.40" />
   <xacro:property name="base_width" value="0.30" />
@@ -26,7 +23,5 @@
   </xacro:property>
   <!-- <xacro:property name="depth_sensor_pose">
-  <!-- <xacro:property name="depth_sensor_pose">
     <origin xyz="0.14 0.0 0.045" rpy="0 0 0"/>
   </xacro:property> -->
-  </xacro:property> -->
 </robot>

File: linorobot2_description/urdf/controllers/diff_drive.urdf.xacro (robot description, xacro)
@@ -1,3 +1,2 @@
-<?xml version="1.0"?>
 <robot xmlns:xacro="http://ros.org/wiki/xacro">
   <xacro:macro name="diff_drive_controller" params="wheel_separation wheel_radius wheel_torque">
@@ -17,6 +16,5 @@
         <publish_odom_tf>false</publish_odom_tf>
         <publish_wheel_tf>true</publish_wheel_tf>
-        <odemetry_topic>/odom</odemetry_topic>
-        <odometry_frame>/odom</odometry_frame>
+        <odometry_frame>odom</odometry_frame>
       </plugin>
     </gazebo>

File: linorobot2_description/urdf/mech/layer2.urdf.xacro (robot description, xacro)
@@ -1,12 +1,9 @@
 <?xml version="1.0"?>
 <robot xmlns:xacro="http://ros.org/wiki/xacro">
-  <xacro:macro name="layer2" params="length width height mass wheel_radius wheel_pos_z">
   <xacro:macro name="layer2" params="length width height mass wheel_radius wheel_pos_z">
    <link name="layer_2">
       <visual>
         <origin xyz="0 -0.0015 0" rpy="0 0 0"/>
-        <origin xyz="0 -0.0015 0" rpy="0 0 0"/>
         <geometry>
-          <box size="${length} ${width} ${height}"/>
           <box size="${length} ${width} ${height}"/>
         </geometry>

File: linorobot2_description/urdf/sensors/depth_sensor.urdf.xacro (robot description, xacro)
@@ -1,3 +1,2 @@
-<?xml version="1.0"?>
 <robot xmlns:xacro="http://ros.org/wiki/xacro">
   <xacro:property name="M_PI" value="3.1415926535897931" />

File: linorobot2_description/urdf/sensors/laser.urdf.xacro (robot description, xacro)
@@ -1,3 +1,2 @@
-<?xml version="1.0"?>
 <robot xmlns:xacro="http://ros.org/wiki/xacro">
   <xacro:property name="M_PI" value="3.1415926535897931" />
