Commit message: .

File: linorobot2_description/urdf/sensors/laser.urdf.xacro (robot description, xacro)
@@ -13,5 +13,5 @@
       </visual>
       <collision>
-        <origin xyz="0 0 -0.025" rpy="0 0 0"/>
+        <origin xyz="0.125 0 0.014" rpy="0 0 0"/>
         <geometry>
           <cylinder radius="0.0375" length="0.05"/>

Commit message: the commit message

File: linorobot2_description/urdf/sensors/laser.urdf.xacro (robot description, xacro)
@@ -4,5 +4,5 @@
     <link name="${frame_id}">
       <visual>
-        <origin xyz="-0.125 0 0.14" rpy="0 0 0"/>
+        <origin xyz="-0.350 0 0.13" rpy="0 0 0"/>
         <geometry>
           <cylinder radius="0.0375" length="0.05"/>
@@ -13,5 +13,5 @@
       </visual>
       <collision>
-        <origin xyz="0.125 0 0.014" rpy="0 0 0"/>
+        <origin xyz="0.350 0 0.013" rpy="0 0 0"/>
         <geometry>
           <cylinder radius="0.0375" length="0.05"/>
